File: AdvancedSTLink.sch (KiCad schematic (older format))
At the start: 51 parts, among them J1 USB_C_Receptacle, J2 Conn_02x03_Odd_Even, J3 Conn_01x06, J4 Conn_01x04, Q1 S8050, SW1 SW_SPDT, SW2 SW_SPDT, U1 STM32F103CBTx, U2 XC6206P332MR, U3 USBLC6-2SC6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

Commit message: Add ESP32 compability.
Parts:
- added R_ESP: DNP, symbol Device:R_Small
- added R_SWD: 0, symbol Device:R_Small
Connections:
- net labels removed: SWD-1.27, Serial-2.54
- wire segments 61 -> 65
Other:
- note added: "For ESP32 / ESP8266: \nPlace R_ESP\n1 - TX\n2 - EN\n5 - GPIO0\n6 - RX\n(From MCU perspective)"
- note added: "For STM32: \nPlace R_SWD\n1 - SWO\n2 - NRST\n5 - SWCLK\n6 - SWDIO"
Changed lines of the file:
@@
 T_SWCLK
 NoConn ~ 3050 2900
-Text GLabel 7550 3050 2    50   Input ~ 0
+Text GLabel 8000 3050 2    50   Input ~ 0
 T_SWDIO
 Text GLabel 6550 3250 0    50   Input ~ 0
@@
 L Connector_Generic:Conn_01x04 J4
 U 1 1 5EA79A78
-P 9400 3350
-F 0 "J4" H 9480 3342 50  0000 L CNN
-F 1 "Conn_01x04" H 9480 3251 50  0000 L CNN
-F 2 "" H 9400 3350 50  0001 C CNN
-F 3 "~" H 9400 3350 50  0001 C CNN
-	1    9400 3350
+P 9400 1450
+F 0 "J4" H 9480 1442 50  0000 L CNN
+F 1 "Conn_01x04" H 9480 1351 50  0000 L CNN
+F 2 "" H 9400 1450 50  0001 C CNN
+F 3 "~" H 9400 1450 50  0001 C CNN
+	1    9400 1450
 	1    0    0    -1
 $EndComp
@@
 L power:GND #PWR041
 U 1 1 5EA7A40A
-P 9200 3250
-F 0 "#PWR041" H 9200 3000 50  0001 C CNN
-F 1 "GND" V 9205 3122 50  0000 R CNN
-F 2 "" H 9200 3250 50  0001 C CNN
-F 3 "" H 9200 3250 50  0001 C CNN
-	1    9200 3250
-	0    1    1    0
-$EndComp
-Text GLabel 9200 3350 0    50   Input ~ 0
+P 9200 1350
+F 0 "#PWR041" H 9200 1100 50  0001 C CNN
+F 1 "GND" V 9205 1222 50  0000 R CNN
+F 2 "" H 9200 1350 50  0001 C CNN
+F 3 "" H 9200 1350 50  0001 C CNN
+	1    9200 1350
+	0    1    1    0
+$EndComp
+Text GLabel 9200 1450 0    50   Input ~ 0
 T_RXD_O
-Text GLabel 9200 3450 0    50   Input ~ 0
+Text GLabel 9200 1550 0    50   Input ~ 0
 T_TXD_O
-Text GLabel 9200 3550 0    50   Input ~ 0
+Text GLabel 9200 1650 0    50   Input ~ 0
 V_OUT_3.3
 $Comp
@@
 	1    0    0    -1
 $EndComp
-Text Label 9500 2200 0    50   ~ 0
-SWD-1.27
-Text Label 9500 3250 0    50   ~ 0
-Serial-2.54
 Wire Wire Line
 	3550 1600 3650 1600
@@
 	1    0    0    -1
 $EndComp
+Text GLabel 8000 2750 2    50   Input ~ 0
+T_TXD
+$Comp
+L Device:R_Small R_SWD
+U 1 1 5EAB9473
+P 7900 3050
+F 0 "R_SWD" V 7704 3050 50  0000 C CNN
+F 1 "0" V 7795 3050 50  0000 C CNN
+F 2 "" H 7900 3050 50  0001 C CNN
+F 3 "~" H 7900 3050 50  0001 C CNN
+	1    7900 3050
+	0    1    1    0
+$EndComp
+$Comp
+L Device:R_Small R_ESP
+U 1 1 5EAB98EE
+P 7900 2750
+F 0 "R_ESP" V 7704 2750 50  0000 C CNN
+F 1 "DNP" V 7795 2750 50  0000 C CNN
+F 2 "" H 7900 2750 50  0001 C CNN
+F 3 "~" H 7900 2750 50  0001 C CNN
+	1    7900 2750
+	0    1    1    0
+$EndComp
+Wire Wire Line
+	7700 2750 7700 3050
+Wire Wire Line
+	7700 3050 7550 3050
+Connection ~ 7700 3050
+Wire Wire Line
+	7800 3050 7700 3050
+Wire Wire Line
+	7700 2750 7800 2750
+Text Notes 8750 3300 0    50   ~ 0
+For STM32: \nPlace R_SWD\n1 - SWO\n2 - NRST\n5 - SWCLK\n6 - SWDIO
+Text Notes 8750 3950 0    50   ~ 0
+For ESP32 / ESP8266: \nPlace R_ESP\n1 - TX\n2 - EN\n5 - GPIO0\n6 - RX\n(From MCU perspective)
 $EndSCHEMATC

Commit message: Update JLink
Parts:
- removed J4: Conn_01x04, symbol Connector_Generic:Conn_01x04
- removed Q1: S8050, Package_TO_SOT_THT:TO-92_Inline, symbol Transistor_BJT:S8050
- removed R1, R11: 100, symbol Device:R_Small
- removed R10: 36k, symbol Device:R_Small
- removed R12: 10k, symbol Device:R_Small
- removed R13: 1.5k, symbol Device:R_Small
- removed R6: 2.2k, symbol Device:R_Small
- removed R_ESP: DNP, symbol Device:R_Small
- removed R_SWD: 0, symbol Device:R_Small
- removed SW2: SW_SPDT, symbol Switch:SW_SPDT
- removed U1: STM32F103CBTx, Package_QFP:LQFP-48_7x7mm_P0.5mm, symbol MCU_ST_STM32F1:STM32F103CBTx
- removed U5, U6, U7: USBLC6-2SC6, Package_TO_SOT_SMD:SOT-23-6, symbol Power_Protection:USBLC6-2SC6
- added C? (x2): 2.2uF, symbol Device:C_Small
- added R? (x7): 220, symbol Device:R_Small
- added U?: STM32F205RETx, Package_QFP:LQFP-64_10x10mm_P0.5mm, symbol MCU_ST_STM32F2:STM32F205RETx
- added U? (x2): USBLC6-2SC6, Package_TO_SOT_SMD:SOT-23-6, symbol Power_Protection:USBLC6-2SC6
- R3: value DNP -> 10k
- R7, R8: value 2.7k -> 2.2k
Connections:
- net labels added: LED1, LED2, RST1, RST2, TCK1, TCK2, TDO, TMS1, TMS2, T_SWO_O
- net labels removed: LED, T_DBG, T_DBG_O, T_NRST, T_RXD, T_RXD_O, T_SWCLK, T_SWDIO, T_SWO, T_TXD, T_TXD_O, USB_RENUMn
- wire segments 65 -> 79
- no-connect marks 16 -> 32
Other:
- note removed: "For ESP32 / ESP8266: \nPlace R_ESP\n1 - TX\n2 - EN\n5 - GPIO0\n6 - RX\n(From MCU perspective)"
- moved on the sheet: C1, C10, C11, C2, C3, C4, C5, C8, C9, D1, D2, J1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

Commit message: ESD diodes
Parts:
- removed U? (x2): USBLC6-2SC6, Package_TO_SOT_SMD:SOT-23-6, symbol Power_Protection:USBLC6-2SC6
- added U? (x2): USBLC6-2P6, Package_TO_SOT_SMD:SOT-666, symbol Power_Protection:USBLC6-2SC6
- U3: value USBLC6-2SC6 -> USBLC6-2P6; footprint Package_TO_SOT_SMD:SOT-23-6 -> Package_TO_SOT_SMD:SOT-666
Changed lines of the file:
@@
 P 2850 5900
 F 0 "U3" V 3000 6250 50  0000 L CNN
-F 1 "USBLC6-2SC6" V 3100 6250 50  0000 L CNN
-F 2 "Package_TO_SOT_SMD:SOT-23-6" H 2100 6300 50  0001 C CNN
+F 1 "USBLC6-2P6" V 3100 6250 50  0000 L CNN
+F 2 "Package_TO_SOT_SMD:SOT-666" H 2100 6300 50  0001 C CNN
 F 3 "http://www2.st.com/resource/en/datasheet/CD00050750.pdf" H 3050 6250 50  0001 C CNN
 	1    2850 5900
@@
 NoConn ~ 3350 3900
 NoConn ~ 3350 4100
-$Comp
-L Power_Protection:USBLC6-2SC6 U?
-U 1 1 5ECDEAB0
-P 7100 3900
-F 0 "U?" V 7250 4250 50  0000 L CNN
-F 1 "USBLC6-2SC6" V 7350 4250 50  0000 L CNN
-F 2 "Package_TO_SOT_SMD:SOT-23-6" H 6350 4300 50  0001 C CNN
-F 3 "http://www2.st.com/resource/en/datasheet/CD00050750.pdf" H 7300 4250 50  0001 C CNN
-	1    7100 3900
-	1    0    0    -1
-$EndComp
 Text GLabel 6600 4000 0    50   Input ~ 0
 T_SWCLK_O
@@
 Wire Wire Line
 	7650 3800 7600 3800
-$Comp
-L Power_Protection:USBLC6-2SC6 U?
-U 1 1 5ECF2C2A
-P 7100 2250
-F 0 "U?" V 7250 2600 50  0000 L CNN
-F 1 "USBLC6-2SC6" V 7350 2600 50  0000 L CNN
-F 2 "Package_TO_SOT_SMD:SOT-23-6" H 6350 2650 50  0001 C CNN
-F 3 "http://www2.st.com/resource/en/datasheet/CD00050750.pdf" H 7300 2600 50  0001 C CNN
-	1    7100 2250
-	1    0    0    -1
-$EndComp
 Text GLabel 6600 2350 0    50   Input ~ 0
 T_NRST_O
@@
 	0    1    1    0
 $EndComp
+$Comp
+L Power_Protection:USBLC6-2SC6 U?
+U 1 1 5EC4CDD1
+P 7100 3900
+F 0 "U?" V 7250 4250 50  0000 L CNN
+F 1 "USBLC6-2P6" V 7350 4250 50  0000 L CNN
+F 2 "Package_TO_SOT_SMD:SOT-666" H 6350 4300 50  0001 C CNN
+F 3 "http://www2.st.com/resource/en/datasheet/CD00050750.pdf" H 7300 4250 50  0001 C CNN
+	1    7100 3900
+	1    0    0    -1
+$EndComp
+$Comp
+L Power_Protection:USBLC6-2SC6 U?
+U 1 1 5EC4E277
+P 7100 2250
+F 0 "U?" V 7250 2600 50  0000 L CNN
+F 1 "USBLC6-2P6" V 7350 2600 50  0000 L CNN
+F 2 "Package_TO_SOT_SMD:SOT-666" H 6350 2650 50  0001 C CNN
+F 3 "http://www2.st.com/resource/en/datasheet/CD00050750.pdf" H 7300 2600 50  0001 C CNN
+	1    7100 2250
+	1    0    0    -1
+$EndComp
+$Comp
+L power:GND #PWR?
+U 1 1 5EC4FB61
+P 7100 4400
+F 0 "#PWR?" H 7100 4150 50  0001 C CNN
+F 1 "GND" V 7105 4272 50  0000 R CNN
+F 2 "" H 7100 4400 50  0001 C CNN
+F 3 "" H 7100 4400 50  0001 C CNN
+	1    7100 4400
+	1    0    0    -1
+$EndComp
+$Comp
+L power:GND #PWR?
+U 1 1 5EC4FE17
+P 7100 2750
+F 0 "#PWR?" H 7100 2500 50  0001 C CNN
+F 1 "GND" V 7105 2622 50  0000 R CNN
+F 2 "" H 7100 2750 50  0001 C CNN
+F 3 "" H 7100 2750 50  0001 C CNN
+	1    7100 2750
+	1    0    0    -1
+$EndComp
+$Comp
+L power:+3.3V #PWR?
+U 1 1 5EC5050A
+P 7100 1750
+F 0 "#PWR?" H 7100 1600 50  0001 C CNN
+F 1 "+3.3V" V 7115 1878 50  0000 L CNN
+F 2 "" H 7100 1750 50  0001 C CNN
+F 3 "" H 7100 1750 50  0001 C CNN
+	1    7100 1750
+	1    0    0    -1
+$EndComp
+$Comp
+L power:+3.3V #PWR?
+U 1 1 5EC50C97
+P 7100 3400
+F 0 "#PWR?" H 7100 3250 50  0001 C CNN
+F 1 "+3.3V" V 7115 3528 50  0000 L CNN
+F 2 "" H 7100 3400 50  0001 C CNN
+F 3 "" H 7100 3400 50  0001 C CNN
+	1    7100 3400
+	1    0    0    -1
+$EndComp
 $EndSCHEMATC

Commit message: remove redundant tvs, layout
Parts:
- removed D?: SMAJ5.0A, symbol Device:D_TVS
- removed Y1: DSX321G 8MHz, symbol Device:Crystal
- added FB1: Ferrite_Bead_Small, Inductor_SMD:L_0603_1608Metric, symbol Device:Ferrite_Bead_Small
- added Y1: DXS321G 8MHz, Crystal:Crystal_SMD_3225-4Pin_3.2x2.5mm, symbol Device:Crystal_GND24_Small
- C1, C10, C11, C12, C2, C3, C4, C5, C6, C7, C8, C9: footprint (none) -> Capacitor_SMD:C_0603_1608Metric
- C13, C14: renamed from C?; footprint (none) -> Capacitor_SMD:C_0603_1608Metric
- D1, D2, D5: footprint (none) -> LED_SMD:LED_0603_1608Metric_Pad1.05x0.95mm_HandSolder
- D3: value B230 -> B230A; footprint Diode_SMD:D_SMB -> Diode_SMD:D_SMA
- J1: footprint (none) -> Connector_USB:USB_C_Receptacle_HRO_TYPE-C-31-M-12
- J2: footprint (none) -> Connector_PinHeader_1.27mm:PinHeader_2x03_P1.27mm_Vertical
- J3: footprint (none) -> Connector_Molex:Molex_CLIK-Mate_502382-0670_1x06-1MP_P1.25mm_Vertical
- L1: footprint (none) -> Inductor_SMD:L_TDK_NLV25_2.5x2.0mm
- R1, R10, R11, R12, R13, R18, R6: renamed from R?; footprint (none) -> Resistor_SMD:R_0603_1608Metric
- R14, R15, R16, R17, R2, R3, R4, R5, R7, R8, R9: footprint (none) -> Resistor_SMD:R_0603_1608Metric
- SW1: footprint (none) -> Button_Switch_SMD:SW_SPDT_CK-JS102011SAQN
- U4: footprint (none) -> Package_TO_SOT_SMD:SOT-23-6
- gave numbers to parts that had none: 3
Connections:
- wire segments 79 -> 85

Commit message: fabrication version
Connections:
- net RST1: now also R1.2
- net RST2: now also R6.2
- net TCK1: no longer R1.2
- net TCK2: no longer R6.2
Changed lines of the file:
@@
 Text GLabel 6600 2350 0    50   Input ~ 0
 T_NRST_O
-Text GLabel 6200 1950 0    50   Input ~ 0
-TCK1
-Text GLabel 6200 2150 0    50   Input ~ 0
-TCK2
 $Comp
 L Device:R_Small R6
@@
 Wire Wire Line
 	2200 4800 2450 4800
+Text GLabel 6200 2150 0    50   Input ~ 0
+RST2
+Text GLabel 6200 1950 0    50   Input ~ 0
+RST1
 $EndSCHEMATC

Commit message: Rev 2
Parts:
- removed R10, R11, R12, R13, R18, R6: 220, Resistor_SMD:R_0603_1608Metric, symbol Device:R_Small
- added D6: LED_Blue, LED_SMD:LED_0603_1608Metric_Pad1.05x0.95mm_HandSolder, symbol Device:LED
- added D7: SS34, lc:SMA(DO-214AC)_S1, symbol Diode:B230
- added J4: Conn_02x03_Odd_Even, Connector_PinHeader_1.27mm:PinHeader_2x03_P1.27mm_Vertical, symbol Connector_Generic:Conn_02x03_Odd_Even
- added RN1, RN2: 220×4, lc:0402_RX4, symbol Device:R_Pack04
- C1, C2: value 10pF -> 12pF; footprint Capacitor_SMD:C_0603_1608Metric -> Capacitor_SMD:C_0402_1005Metric
- C10, C11, C13, C14, C3, C4, C5, C7, C8, C9: footprint Capacitor_SMD:C_0603_1608Metric -> Capacitor_SMD:C_0402_1005Metric
- D3: value B230A -> SS34; footprint Diode_SMD:D_SMA -> lc:SMA(DO-214AC)_S1
- D4: footprint Diode_SMD:D_SOD-123 -> lc:SOD-123
- R1: value 220 -> 39k; footprint Resistor_SMD:R_0603_1608Metric -> Resistor_SMD:R_0402_1005Metric
- R14, R15, R17, R2, R4, R5, R7, R8: footprint Resistor_SMD:R_0603_1608Metric -> Resistor_SMD:R_0402_1005Metric
- R16: value 1.5k -> 1.8k; footprint Resistor_SMD:R_0603_1608Metric -> Resistor_SMD:R_0402_1005Metric
- R9: value 330k -> 2.2k; footprint Resistor_SMD:R_0603_1608Metric -> Resistor_SMD:R_0402_1005Metric
- U2: footprint Package_TO_SOT_SMD:SOT-23 -> lc:SOT-23-3L
- U3, U5, U6: symbol Power_Protection:USBLC6-2SC6 -> AdvancedSTLink-rescue:USBLC6-2SC6-Power_Protection
- U4: footprint Package_TO_SOT_SMD:SOT-23-6 -> lc:SOT-23-6
- Y1: value DXS321G 8MHz -> NX3225GA-12MHz
Connections:
- net +3V3: now also R9.1
- net GND: now also SW1.3 (C), D6.1 (K), J4.2 (Pin_2); no longer SW1.1 (A)
- net RST1: now also RN2.8 (R1.2); no longer R1.2
- net RST2: now also RN2.7 (R2.2)
- net TCK1: now also RN1.8 (R1.2)
- net TCK2: now also RN1.7 (R2.2)
- net TDO: now also RN2.5 (R4.2)
- net TMS1: now also RN1.5 (R4.2)
- net TMS2: now also RN1.6 (R3.2)
- net T_NRST_O: now also J4.3 (Pin_3)
- net T_SWCLK_O: now also J4.4 (Pin_4)
- net T_SWDIO_O: now also J4.6 (Pin_6)
- net T_SWO_O: now also J4.1 (Pin_1)
- net VBUS: now also D7.2 (A); no longer C6.1, R9.1, U4.5 (IN)
- net V_OUT_3.3: now also J4.5 (Pin_5)
- net T_SWDIO_I: now reaches U6.4 (IO2)
- net T_SWDIO_I: now also RN1.3 (R3.1), RN1.4 (R4.1)
- net T_SWCLK_I: now reaches U6.6 (IO1)
- net T_SWCLK_I: now also RN1.1 (R1.1), RN1.2 (R2.1)
- net T_SWO_I: now reaches U5.4 (IO2)
- net T_SWO_I: now also RN2.4 (R4.1)
- net at R1.1: now also U4.4 (EN); no longer U5.6 (IO1)
- new net: C6.1, D7.1 (K), U4.5 (IN)
- new net: R9.2, SW1.1 (A)
- new net: D6.2 (A), R1.2, SW1.2 (B)
- new net T_NRST_I: RN2.1 (R1.1), RN2.2 (R2.1), U5.6 (IO1)
Other:
- moved on the sheet: C1, C10, C11, C12, C13, C14, C2, C3, C4, C5, C6, C7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
